File: FirstdraftKicad.kicad_pcb (KiCad board)
At the start: 2 copper layers, 26 parts, among them J1 Conn_Coaxial, J2 Conn_Coaxial, U1 Opamp_Quad, U2 Diff, U3 ADC, U4 Diff

Commit message: Updated kicad files
Parts:
- removed U1: Opamp_Quad, Package_DIP:DIP-14_W7.62mm
- removed U2, U4: Diff, Package_DFN_QFN:DFN-8-1EP_3x3mm_P0.5mm_EP1.66x2.38mm
- removed U3: ADC, Package_LGA:LGA-16_3x3mm_P0.5mm
- added AD4680BCPZ1: AD4680BCPZ, Package_LGA:LGA-16_3x3mm_P0.5mm, F.Cu at (144.8, 104.1)
- added AD8138: TOP, Package_DFN_QFN:DFN-8-1EP_3x3mm_P0.5mm_EP1.66x2.38mm, F.Cu at (139.7, 88.9)
- added AD8138(2)1: Bottom, Package_DFN_QFN:DFN-8-1EP_3x3mm_P0.5mm_EP1.66x2.38mm, F.Cu at (149.9, 88.9)
- added OPA4228PA1: OPA1604, Package_DIP:DIP-14_W7.62mm, F.Cu at (141.0, 68.6)
- C1, C2, C4: value Cap -> 1µF
- C10, C11, C8, C9: value Cap -> 0.05µF
- C3, C6, C7: value Cap -> 0.1µF
- J1, J2: footprint Connector_Coaxial:BNC_PanelMountable_Vertical -> Connector_Coaxial:MMCX_Molex_73415-1471_Vertical
- R1: value R -> 10.8kΩ
- R2: value R -> 450kΩ
- R3, R4, R5, R6, R7, R8: value R -> 0.5kΩ
- moved A1 98.8 mm to (154.8, 156.2), turned to 180 degrees
- moved J2 75.2 mm to (152.4, 58.4)
- moved J1 53.8 mm to (137.2, 58.4)
- moved C6 45.7 mm to (137.2, 76.2)
- moved C8 44.6 mm to (139.7, 94.0)
- moved R2 43.5 mm to (137.2, 81.3)
- moved R7 41.3 mm to (152.4, 83.8)
- moved R1 40.7 mm to (137.2, 68.6), turned to 90 degrees
- moved C7 39.2 mm to (152.4, 76.2)
- moved R6 33.4 mm to (147.3, 88.9), turned to -90 degrees
- moved R8 33.0 mm to (149.9, 96.5)
- moved C9 32.5 mm to (134.6, 91.4), turned to -90 degrees
- moved C11 31.4 mm to (147.3, 94.0), turned to -90 degrees
- moved C2 30.2 mm to (149.9, 106.7), turned to -90 degrees
- moved R5 28.4 mm to (134.6, 96.5), turned to -90 degrees
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Connections:
- A1 pad 11: unconnected-(A1-Pad11) -> Net-(AD4680BCPZ1-Pad16)
- A1 pad 13: unconnected-(A1-Pad13) -> Net-(AD4680BCPZ1-Pad13)
- A1 pad 22: unconnected-(A1-Pad22) -> Net-(AD4680BCPZ1-Pad14)
- C1 pad 1: Net-(C1-Pad1) -> +3V3
- C10 pad 1: Net-(U4-Pad3) -> +5V
- C10 pad 2: GND -> Net-(AD8138(2)1-Pad3)
- C11 pad 2: GND -> -5V
- C2 pad 1: Net-(U3-Pad3) -> +1V8
- C3 pad 1: Net-(U3-Pad9) -> +2V5
- C4 pad 1: Net-(U3-Pad2) -> +3V3
- C5 pad 1: Net-(U3-Pad11) -> +4V
- C6 pad 1: Net-(U1-Pad4) -> +15V
- C6 pad 2: GND -> Net-(C6-Pad2)
- C7 pad 2: GND -> -15V
- C8 pad 1: Net-(U2-Pad3) -> +5V
- C8 pad 2: GND -> Net-(AD8138-Pad3)
- C9 pad 2: GND -> -5V
Routing:
- net Net-(AD4680BCPZ1-Pad14): track 0.00 -> 36.9 mm, vias 0 -> 2
- net Net-(AD4680BCPZ1-Pad13): track 0.00 -> 32.9 mm
- net Net-(AD4680BCPZ1-Pad16): track 0.00 -> 32.8 mm, vias 0 -> 2
- net Net-(AD8138-Pad8): track 3.41 -> 32.4 mm, vias 0 -> 2
- net +5V: track 0.00 -> 26.9 mm, vias 0 -> 2
- net Net-(AD4680BCPZ1-Pad7): track 0.00 -> 26.8 mm, vias 0 -> 2
- net Net-(J2-Pad1): track 21.4 -> 44.4 mm, vias 0 -> 2
- net Net-(AD4680BCPZ1-Pad6): track 0.00 -> 21.8 mm
- net Net-(AD4680BCPZ1-Pad8): track 3.82 -> 24.5 mm, vias 0 -> 2
- net +3V3: track 0.00 -> 20.1 mm, vias 0 -> 4
- net GND: track 29.3 -> 48.8 mm, vias 0 -> 4
- net Net-(AD4680BCPZ1-Pad5): track 0.00 -> 18.9 mm
- net -5V: track 0.00 -> 18.0 mm, vias 0 -> 2
- net Net-(AD8138-Pad1): track 0.00 -> 13.4 mm
- net Net-(AD8138-Pad6): track 0.00 -> 13.3 mm, vias 0 -> 2
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